File: power.kicad_sch (KiCad schematic)
At the start: 13 parts, among them J11 CONN_12V, J12 Screw_Terminal_01x02, Q2 DMP3037LSS, SW3 PWR_SW, U12 LM2576S-3.3

Commit message: Final annotate pass
Parts:
- renumbered C86 to C601, C87 to C602, C88 to C603, C89 to C604, D1 to D601, D2 to D602, J11 to J601, J12 to J602, L4 to L601, Q2 to Q601, R35 to R601, SW3 to SW601, U12 to U601
Changed lines of the file:
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@@
   (symbol (lib_id "Device:D_Schottky") (at 176.53 85.09 270) (unit 1)
     (in_bom yes) (on_board yes) (fields_autoplaced)
-    (property "Reference" "D1" (id 0) (at 178.562 83.9378 90)
+    (property "Reference" "D601" (id 0) (at 178.562 83.9378 90)
       (effects (font (size 1.27 1.27)) (justify left))
     )
@@
   (symbol (lib_id "Device:L") (at 185.42 77.47 90) (unit 1)
     (in_bom yes) (on_board yes)
-    (property "Reference" "L4" (id 0) (at 185.42 80.01 90))
+    (property "Reference" "L601" (id 0) (at 185.42 80.01 90))
     (property "Value" "68u 5A" (id 1) (at 185.42 74.93 90))
     (property "Footprint" "Inductor_THT:L_Toroid_Vertical_L24.6mm_W15.5mm_P11.44mm_Pulse_KM-4" (id 2) (at 185.42 77.47 0)
@@
   (symbol (lib_id "Connector:Screw_Terminal_01x02") (at 88.9 59.69 180) (unit 1)
     (in_bom yes) (on_board yes) (fields_autoplaced)
-    (property "Reference" "J12" (id 0) (at 88.9 50.8 0))
+    (property "Reference" "J602" (id 0) (at 88.9 50.8 0))
     (property "Value" "Screw_Terminal_01x02" (id 1) (at 88.9 53.34 0))
     (property "Footprint" "TerminalBlock_Phoenix:TerminalBlock_Phoenix_MKDS-1,5-2-5.08_1x02_P5.08mm_Horizontal" (id 2) (at 88.9 59.69 0)
@@
   (symbol (lib_id "Device:C_Polarized") (at 219.71 85.09 0) (unit 1)
     (in_bom yes) (on_board yes) (fields_autoplaced)
-    (property "Reference" "C89" (id 0) (at 222.631 83.3663 0)
+    (property "Reference" "C604" (id 0) (at 222.631 83.3663 0)
       (effects (font (size 1.27 1.27)) (justify left))
     )
@@
   (symbol (lib_id "Connector:Barrel_Jack_MountingPin") (at 87.63 74.93 0) (unit 1)
     (in_bom yes) (on_board yes) (fields_autoplaced)
-    (property "Reference" "J11" (id 0) (at 87.63 67.4202 0))
+    (property "Reference" "J601" (id 0) (at 87.63 67.4202 0))
     (property "Value" "CONN_12V" (id 1) (at 87.63 69.9571 0))
     (property "Footprint" "" (id 2) (at 88.9 75.946 0)
@@
   (symbol (lib_id "power:GND") (at 219.71 91.44 0) (unit 1)
     (in_bom yes) (on_board yes) (fields_autoplaced)
-    (property "Reference" "#PWR058" (id 0) (at 219.71 97.79 0)
+    (property "Reference" "#PWR0608" (id 0) (at 219.71 97.79 0)
       (effects (font (size 1.27 1.27)) hide)
     )
@@
   (symbol (lib_id "power:GND") (at 121.92 87.63 0) (unit 1)
     (in_bom yes) (on_board yes) (fields_autoplaced)
-    (property "Reference" "#PWR050" (id 0) (at 121.92 93.98 0)
+    (property "Reference" "#PWR0602" (id 0) (at 121.92 93.98 0)
       (effects (font (size 1.27 1.27)) hide)
     )
@@
   (symbol (lib_id "power:GND") (at 229.87 102.87 0) (unit 1)
     (in_bom yes) (on_board yes) (fields_autoplaced)
-    (property "Reference" "#PWR056" (id 0) (at 229.87 109.22 0)
+    (property "Reference" "#PWR0609" (id 0) (at 229.87 109.22 0)
       (effects (font (size 1.27 1.27)) hide)
     )
@@
   (symbol (lib_id "power:GND") (at 194.31 91.44 0) (unit 1)
     (in_bom yes) (on_board yes) (fields_autoplaced)
-    (property "Reference" "#PWR054" (id 0) (at 194.31 97.79 0)
+    (property "Reference" "#PWR0606" (id 0) (at 194.31 97.79 0)
       (effects (font (size 1.27 1.27)) hide)
     )
@@
   (symbol (lib_id "power:GND") (at 130.81 87.63 0) (unit 1)
     (in_bom yes) (on_board yes) (fields_autoplaced)
-    (property "Reference" "#PWR051" (id 0) (at 130.81 93.98 0)
+    (property "Reference" "#PWR0603" (id 0) (at 130.81 93.98 0)
       (effects (font (size 1.27 1.27)) hide)
     )
@@
   (symbol (lib_id "power:VDD") (at 232.41 77.47 270) (unit 1)
     (in_bom yes) (on_board yes) (fields_autoplaced)
-    (property "Reference" "#PWR057" (id 0) (at 228.6 77.47 0)
+    (property "Reference" "#PWR0610" (id 0) (at 228.6 77.47 0)
       (effects (font (size 1.27 1.27)) hide)
     )
@@
   (symbol (lib_id "power:GND") (at 149.86 87.63 0) (unit 1)
     (in_bom yes) (on_board yes) (fields_autoplaced)
-    (property "Reference" "#PWR052" (id 0) (at 149.86 93.98 0)
+    (property "Reference" "#PWR0604" (id 0) (at 149.86 93.98 0)
       (effects (font (size 1.27 1.27)) hide)
     )
@@
   (symbol (lib_id "Device:C_Polarized") (at 130.81 80.01 0) (unit 1)
     (in_bom yes) (on_board yes) (fields_autoplaced)
-    (property "Reference" "C86" (id 0) (at 133.731 78.2863 0)
+    (property "Reference" "C601" (id 0) (at 133.731 78.2863 0)
       (effects (font (size 1.27 1.27)) (justify left))
     )
@@
   (symbol (lib_id "Switch:SW_SPST") (at 109.22 72.39 0) (unit 1)
     (in_bom yes) (on_board yes) (fields_autoplaced)
-    (property "Reference" "SW3" (id 0) (at 109.22 67.0392 0))
+    (property "Reference" "SW601" (id 0) (at 109.22 67.0392 0))
     (property "Value" "PWR_SW" (id 1) (at 109.22 69.5761 0))
     (property "Footprint" "" (id 2) (at 109.22 72.39 0)
@@
   (symbol (lib_id "Regulator_Switching:LM2576S-3.3") (at 157.48 74.93 0) (unit 1)
     (in_bom yes) (on_board yes) (fields_autoplaced)
-    (property "Reference" "U12" (id 0) (at 157.48 66.1502 0))
+    (property "Reference" "U601" (id 0) (at 157.48 66.1502 0))
     (property "Value" "LM2576S-3.3" (id 1) (at 157.48 68.6871 0))
     (property "Footprint" "Package_TO_SOT_SMD:TO-263-5_TabPin3" (id 2) (at 157.48 81.28 0)
@@
   (symbol (lib_id "Device:LED") (at 229.87 95.25 90) (unit 1)
     (in_bom yes) (on_board yes) (fields_autoplaced)
-    (property "Reference" "D2" (id 0) (at 233.68 95.5674 90)
+    (property "Reference" "D602" (id 0) (at 233.68 95.5674 90)
       (effects (font (size 1.27 1.27)) (justify right))
     )
@@
   (symbol (lib_id "Device:R") (at 229.87 83.82 0) (unit 1)
     (in_bom yes) (on_board yes) (fields_autoplaced)
-    (property "Reference" "R35" (id 0) (at 232.41 82.5499 0)
+    (property "Reference" "R601" (id 0) (at 232.41 82.5499 0)
       (effects (font (size 1.27 1.27)) (justify left))
     )
@@
   (symbol (lib_id "Device:C_Polarized") (at 207.01 85.09 0) (unit 1)
     (in_bom yes) (on_board yes) (fields_autoplaced)
-    (property "Reference" "C88" (id 0) (at 209.931 83.3663 0)
+    (property "Reference" "C603" (id 0) (at 209.931 83.3663 0)
       (effects (font (size 1.27 1.27)) (justify left))
     )
@@
   (symbol (lib_id "power:GND") (at 207.01 91.44 0) (unit 1)
     (in_bom yes) (on_board yes) (fields_autoplaced)
-    (property "Reference" "#PWR055" (id 0) (at 207.01 97.79 0)
+    (property "Reference" "#PWR0607" (id 0) (at 207.01 97.79 0)
       (effects (font (size 1.27 1.27)) hide)
     )
@@
   (symbol (lib_id "power:GND") (at 92.71 87.63 0) (unit 1)
     (in_bom yes) (on_board yes) (fields_autoplaced)
-    (property "Reference" "#PWR049" (id 0) (at 92.71 93.98 0)
+    (property "Reference" "#PWR0601" (id 0) (at 92.71 93.98 0)
       (effects (font (size 1.27 1.27)) hide)
     )
@@
   (symbol (lib_id "Device:C_Polarized") (at 194.31 85.09 0) (unit 1)
     (in_bom yes) (on_board yes) (fields_autoplaced)
-    (property "Reference" "C87" (id 0) (at 198.12 82.9309 0)
+    (property "Reference" "C602" (id 0) (at 198.12 82.9309 0)
       (effects (font (size 1.27 1.27)) (justify left))
     )
@@
   (symbol (lib_id "Transistor_FET:FDS9435A") (at 121.92 74.93 90) (unit 1)
     (in_bom yes) (on_board yes) (fields_autoplaced)
-    (property "Reference" "Q2" (id 0) (at 121.92 64.77 90))
+    (property "Reference" "Q601" (id 0) (at 121.92 64.77 90))
     (property "Value" "DMP3037LSS" (id 1) (at 121.92 67.31 90))
     (property "Footprint" "Package_SO:SOIC-8_3.9x4.9mm_P1.27mm" (id 2) (at 123.825 69.85 0)
@@
   (symbol (lib_id "power:GND") (at 176.53 91.44 0) (unit 1)
     (in_bom yes) (on_board yes) (fields_autoplaced)
-    (property "Reference" "#PWR053" (id 0) (at 176.53 97.79 0)
-      (effects (font (size 1.27 1.27)) hide)
-    )
+    (property "Reference" "#PWR0605" (id 0) (at 176.53 97.79 0)
+      (effects (font (size 1.27 1.27)) hide)
+    )

Commit message: More footprints
Parts:
- J601: footprint (none) -> Connector_BarrelJack:BarrelJack_CUI_PJ-063AH_Horizontal; Part (none) -> 490-PJ-063AH
Changed lines of the file:
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@@
     (property "Reference" "J601" (id 0) (at 87.63 67.4202 0))
     (property "Value" "CONN_12V" (id 1) (at 87.63 69.9571 0))
-    (property "Footprint" "" (id 2) (at 88.9 75.946 0)
+    (property "Footprint" "Connector_BarrelJack:BarrelJack_CUI_PJ-063AH_Horizontal" (id 2) (at 88.9 75.946 0)
       (effects (font (size 1.27 1.27)) hide)
     )
@@
       (effects (font (size 1.27 1.27)) hide)
     )
+    (property "Part" "490-PJ-063AH" (id 4) (at 87.63 74.93 0)
+      (effects (font (size 1.27 1.27)) hide)
+    )
