File: ram.kicad_sch (KiCad schematic)
At the start: 56 parts, among them U401 IS42S86400D, U402 IS42S86400D, U403 IS42S86400D, U404 IS42S86400D, U405 IS42S86400D, U406 IS42S86400D, U407 IS42S86400D, U408 IS42S86400D

Commit message: Fully update PCB and schematic after BOM consolidation
Parts:
- C401, C402, C403, C404, C405, C406, C407, C408, C409, C410, C411, C412, C413, C414, C415, C416, C417, C418, C419, C420, C421, C422, C423, C424, C425, C426, C427, C428, C429, C430, C431, C432, C433, C434, C435, C436, C437, C438, C439, C440, C441, C442, C443, C444, C445, C446, C447, C448: Part (none) -> 603-CC603ZRY5V7BB104
- U401, U402, U403, U404, U405, U406, U407, U408: Part (none) -> 870-IS42S86400D-7TLI
